File: pcb/Nu2031.brd (EAGLE design)
At the start: 30.5 x 50.8 mm, 26 parts, among them IC1 6522P-ST, IC2 75160SO, IC3 75161SO, IC4 XC9572XLVQG64, X2 2520-

Commit message: First working config
* Fix some of the IEEE logic in HDL
* Add resistor to ROM selection, to default to IEC
* Add patched 1541 (2031-ish) DOS
Parts:
- added R3: (no value), resistor:R0402
- moved ROM 48.3 mm to (29.2, 1.27)
Connections:
- net ROM_SEL: now also R3.1
- net VCC: now also R3.2
Routing:
- net VCC: track 73.9 -> 95.9 mm
- net ROM_SEL: track 39.0 -> 42.8 mm
Changed lines of the file:
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@@
 <wire x1="30.48" y1="1.27" x2="30.48" y2="49.53" width="0" layer="20"/>
 <wire x1="30.48" y1="49.53" x2="29.21" y2="50.8" width="0" layer="20" curve="90"/>
-<text x="22.86" y="46.99" size="1.27" layer="27" ratio="10">GND</text>
+<text x="22.86" y="2.54" size="1.27" layer="27" ratio="10">GND</text>
+<dimension x1="1.27" y1="50.8" x2="1.27" y2="0" x3="-1.27" y3="25.4" textsize="1.778" layer="48"/>
+<dimension x1="0" y1="49.53" x2="30.48" y2="49.53" x3="15.24" y3="52.07" textsize="1.778" layer="48"/>
 </plain>
 <attributes>
@@
 <attribute name="VALUE" x="6.985" y="33.9725" size="1.27" layer="28" rot="MR0"/>
 </element>
-<element name="ROM" library="testpad" package="B1,27" value="PTR1B1,27" x="29.21" y="49.53" smashed="yes">
-<attribute name="TP_SIGNAL_NAME" value="" x="28.575" y="47.625" size="1" layer="37"/>
-<attribute name="NAME" x="26.3525" y="47.0535" size="1.27" layer="25" ratio="10"/>
+<element name="ROM" library="testpad" package="B1,27" value="PTR1B1,27" x="29.21" y="1.27" smashed="yes">
+<attribute name="TP_SIGNAL_NAME" value="" x="28.575" y="-0.635" size="1" layer="37"/>
+<attribute name="NAME" x="26.3525" y="2.6035" size="1.27" layer="25" ratio="10"/>
 </element>
 <element name="T1" library="transistor" package="SOT23-BEC" value="" x="13.0175" y="10.795" smashed="yes" rot="MR90">
@@
 <attribute name="TP_SIGNAL_NAME" value="" x="1.27" y="15.875" size="1" layer="38" rot="MR0"/>
 <attribute name="NAME" x="5.08" y="17.145" size="1.27" layer="26" rot="MR0"/>
+</element>
+<element name="R3" library="resistor" package="R0402" value="" x="27.94" y="5.08" smashed="yes" rot="R180">
+<attribute name="NAME" x="24.4475" y="4.445" size="1.27" layer="25"/>
+<attribute name="VALUE" x="28.575" y="6.985" size="1.27" layer="27" rot="R180"/>
 </element>
 </elements>
@@
 <via x="5.08" y="33.02" extent="1-16" drill="0.3048"/>
 <via x="15.875" y="16.8275" extent="1-16" drill="0.3048"/>
-<via x="24.13" y="49.53" extent="1-16" drill="1"/>
+<via x="24.13" y="1.27" extent="1-16" drill="1"/>
 <contactref element="T1" pad="E"/>
 <contactref element="T2" pad="E"/>
@@
 <wire x1="6.985" y1="30.1625" x2="11.7475" y2="25.4" width="0.3048" layer="1"/>
 <wire x1="11.7475" y1="25.4" x2="11.7475" y2="23.8125" width="0.3048" layer="1"/>
-<wire x1="11.7475" y1="23.8125" x2="12.7" y2="22.86" width="0.3048" layer="1"/>
-<wire x1="12.7" y1="22.86" x2="13.0175" y2="22.5425" width="0.3048" layer="1"/>
+<wire x1="11.7475" y1="23.8125" x2="13.0175" y2="22.5425" width="0.3048" layer="1"/>
 <wire x1="13.0175" y1="22.5425" x2="14.605" y2="20.955" width="0.3048" layer="1"/>
 <wire x1="14.605" y1="20.955" x2="15.24" y2="20.955" width="0.3048" layer="1"/>
@@
 <wire x1="8.57" y1="34.925" x2="8.57" y2="33.02" width="0.3048" layer="16"/>
 <wire x1="2.54" y1="1.27" x2="6.35" y2="1.27" width="0.3048" layer="1"/>
-<wire x1="6.35" y1="1.27" x2="6.35" y2="4.3942" width="0.3048" layer="1"/>
+<wire x1="6.35" y1="1.27" x2="6.35" y2="2.54" width="0.3048" layer="1"/>
+<wire x1="6.35" y1="2.54" x2="6.35" y2="4.3942" width="0.3048" layer="1"/>
 <wire x1="7" y1="35.8775" x2="7" y2="34.94" width="0.3048" layer="16"/>
 <wire x1="7" y1="34.94" x2="6.985" y2="34.925" width="0.3048" layer="16"/>
@@
 <wire x1="7.62" y1="17.145" x2="13.0175" y2="22.5425" width="0.1524" layer="16"/>
 <via x="13.0175" y="22.5425" extent="1-16" drill="0.3048"/>
+<contactref element="R3" pad="2"/>
+<wire x1="27.29" y1="5.08" x2="24.75" y2="2.54" width="0.1524" layer="1"/>
+<wire x1="24.75" y1="2.54" x2="6.35" y2="2.54" width="0.1524" layer="1"/>
 </signal>
 <signal name="DATA_IN">
@@
 <signal name="ROM_SEL">
 <contactref element="ROM" pad="TP"/>
-<via x="29.21" y="49.53" extent="1-16" drill="1"/>
-<via x="26.67" y="49.53" extent="1-16" drill="1"/>
-<wire x1="29.845" y1="26.67" x2="29.845" y2="48.895" width="0.1524" layer="1"/>
-<wire x1="29.845" y1="48.895" x2="29.21" y2="49.53" width="0.1524" layer="1"/>
-<wire x1="29.21" y1="49.53" x2="26.67" y2="49.53" width="0.1524" layer="1"/>
+<via x="29.21" y="1.27" extent="1-16" drill="1"/>
+<via x="26.67" y="1.27" extent="1-16" drill="1"/>
+<wire x1="29.845" y1="26.67" x2="29.845" y2="5.08" width="0.1524" layer="1"/>
+<wire x1="29.845" y1="5.08" x2="29.845" y2="1.905" width="0.1524" layer="1"/>
+<wire x1="29.845" y1="1.905" x2="29.21" y2="1.27" width="0.1524" layer="1"/>
+<wire x1="29.21" y1="1.27" x2="26.67" y2="1.27" width="0.1524" layer="1"/>
 <contactref element="IC4" pad="57"/>
 <wire x1="17.13" y1="25.65" x2="17.8475" y2="25.65" width="0.1524" layer="1"/>
@@
 <wire x1="18.0975" y1="25.4" x2="28.575" y2="25.4" width="0.1524" layer="1"/>
 <wire x1="28.575" y1="25.4" x2="29.845" y2="26.67" width="0.1524" layer="1"/>
+<contactref element="R3" pad="1"/>
+<wire x1="28.59" y1="5.08" x2="29.845" y2="5.08" width="0.1524" layer="1"/>
 </signal>
 <signal name="N$3">

Commit message: Implement auto-reset functionality and clean up Verilog a bit.
Routing:
- net ROM_SEL: track 42.8 -> 40.3 mm
Changed lines of the file:
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@@
 <via x="29.21" y="1.27" extent="1-16" drill="1"/>
 <via x="26.67" y="1.27" extent="1-16" drill="1"/>
-<wire x1="29.845" y1="26.67" x2="29.845" y2="5.08" width="0.1524" layer="1"/>
+<wire x1="29.845" y1="24.13" x2="29.845" y2="5.08" width="0.1524" layer="1"/>
 <wire x1="29.845" y1="5.08" x2="29.845" y2="1.905" width="0.1524" layer="1"/>
 <wire x1="29.845" y1="1.905" x2="29.21" y2="1.27" width="0.1524" layer="1"/>
@@
 <wire x1="17.8475" y1="25.65" x2="18.0975" y2="25.4" width="0.1524" layer="1"/>
 <wire x1="18.0975" y1="25.4" x2="28.575" y2="25.4" width="0.1524" layer="1"/>
-<wire x1="28.575" y1="25.4" x2="29.845" y2="26.67" width="0.1524" layer="1"/>
+<wire x1="28.575" y1="25.4" x2="29.845" y2="24.13" width="0.1524" layer="1"/>
 <contactref element="R3" pad="1"/>
 <wire x1="28.59" y1="5.08" x2="29.845" y2="5.08" width="0.1524" layer="1"/>
